Commit message: feat(elexhub): refine model and add webcam setup
Match the owner-confirmed black metal kit in shared CAD and simulation exports, retain provisional dimensions and disabled physical commissioning, and preserve missing-feed detection.

Add operator-started ChArUco capture and intrinsics calibration with image integrity checks, keep raw preview separate from registered robot observations, and retain component research and reproducible validation evidence.

Validation: 64 Elexhub, camera and driver tests passed; lint and browser layout checks passed; CAD/export identities and bundle hashes verified. Real arm measurements, camera calibration and physical trials remain pending.

File: assets/elexhub/provisional/elexhub.urdf (robot description, URDF)
Before this commit: robot elexhub_provisional, 9 links, 8 joints
Links:
- link base_link: geometry visual mesh filename=meshes/base__anodized.obj; visual mesh filename=meshes/base__cap.obj
- link finger_left: geometry collision box size=0.018 0.006 0.065; visual mesh filename=meshes/finger_left__anodized.obj
- link finger_right: geometry collision box size=0.018 0.006 0.065; visual mesh filename=meshes/finger_right__anodized.obj
- link forearm: geometry collision box size=0.032 0.028 0.1; visual mesh filename=meshes/forearm__anodized.obj
- link tool: geometry collision box size=0.04 0.03 0.025; visual mesh filename=meshes/tool__anodized.obj
- link turret: geometry collision box size=0.045 0.04 0.055; visual mesh filename=meshes/turret__anodized.obj
- link upper_arm: geometry collision box size=0.038 0.028 0.105; visual mesh filename=meshes/upper_arm__anodized.obj
- link wrist: geometry collision box size=0.038 0.035 0.045; visual mesh filename=meshes/wrist__anodized.obj
Joints:
- joint finger_left: limit lower=0 upper=0.0175 effort=3 velocity=.03 -> lower=0 upper=0.0275 effort=3 velocity=.03; origin xyz=0 -0.0205 0.025 -> xyz=0 -0.0305 0.025
- joint finger_right: limit lower=0 upper=0.0175 effort=3 velocity=.03 -> lower=0 upper=0.0275 effort=3 velocity=.03; origin xyz=0 0.0205 0.025 -> xyz=0 0.0305 0.025
- joint tcp_fixed: origin xyz=0 0 0.0535 -> xyz=0 0 0.07375

Commit message: Add photo-based Elexhub model and hand mirroring
Refine the arm from the owner's five photos and provide matching editable
CAD, material meshes, robot-only MuJoCo export, viewer and measured-input
guide. Preserve provisional dimensions and the existing joint topology.

Add local left-hand detection and relative gripper steering with pinch
control, bounded simulation steps, loss holding, camera ownership and
explicit start/stop controls. Load reviewed assets without rebuilding them
on console startup and document the persistent local launcher.

Validation: 117 relevant tests passed across the model, camera and control
suites. The synthetic hand sweep moved all three axes with zero rejected
steps; live webcam preview and Start/Hold/Off were exercised. Reviewed
artifact hashes and protected profiles/evaluation files remain unchanged.

File: assets/elexhub/provisional/elexhub.urdf (robot description, URDF)
Before this commit: robot elexhub_provisional, 9 links, 8 joints
Links:
- link base_link: geometry visual mesh filename=meshes/base__anodized.obj; visual mesh filename=meshes/base__brown.obj
